Commit message: modified the URDF

File: src/robot_arm_urdf/urdf/robot_arm_urdf.urdf (robot description, URDF)
Before this commit: robot robot_arm_urdf, 9 links, 8 joints
Joints:
- joint joint_4: limit lower=0 upper=-3.142 effort=200 velocity=3 -> lower=-3.142 upper=0 effort=200 velocity=3

Commit message: code is broken, will make a new build later.

File: src/robot_arm_urdf/urdf/robot_arm_urdf.urdf (robot description, URDF)
Before this commit: robot robot_arm_urdf, 9 links, 8 joints
Links:
- link base_link: geometry collision mesh filename=package://robot_arm_urdf/meshes/base_link.STL scale=0.001 0.001 0.001; visual mesh filename=package://robot_arm_urdf/meshes/base_link.STL scale=0.001 0.001 0.001
- link link_1: geometry collision mesh filename=package://robot_arm_urdf/meshes/link_1.STL scale=0.001 0.001 0.001; visual mesh filename=package://robot_arm_urdf/meshes/link_1.STL scale=0.001 0.001 0.001
- link link_2: geometry collision mesh filename=package://robot_arm_urdf/meshes/link_2.STL scale=0.001 0.001 0.001; visual mesh filename=package://robot_arm_urdf/meshes/link_2.STL scale=0.001 0.001 0.001
- link link_3: geometry collision mesh filename=package://robot_arm_urdf/meshes/link_3.STL scale=0.001 0.001 0.001; visual mesh filename=package://robot_arm_urdf/meshes/link_3.STL scale=0.001 0.001 0.001
- link link_4: geometry collision mesh filename=package://robot_arm_urdf/meshes/link_4.STL scale=0.001 0.001 0.001; visual mesh filename=package://robot_arm_urdf/meshes/link_4.STL scale=0.001 0.001 0.001
- link link_5: geometry collision mesh filename=package://robot_arm_urdf/meshes/link_5.STL scale=0.001 0.001 0.001; visual mesh filename=package://robot_arm_urdf/meshes/link_5.STL scale=0.001 0.001 0.001
- link link_6: geometry collision mesh filename=package://robot_arm_urdf/meshes/link_6.STL scale=0.001 0.001 0.001; visual mesh filename=package://robot_arm_urdf/meshes/link_6.STL scale=0.001 0.001 0.001
- link link_7: geometry collision mesh filename=package://robot_arm_urdf/meshes/link_7.STL scale=0.001 0.001 0.001; visual mesh filename=package://robot_arm_urdf/meshes/link_7.STL scale=0.001 0.001 0.001
